File: Alimentacion.sch (KiCad schematic (older format))
At the start: 10 parts, among them J7 Batería2, J8 Bateria1, U11 LM2596S-5, U12 AMS1117-3.3

Commit message: Placa terminada
Parts:
- added NT1: Net-Tie_2, NetTie:NetTie-2_SMD_Pad2.0mm, symbol Device:Net-Tie_2
- renumbered J7 to J13, J8 to J14, U11 to U5, U12 to U6
Connections:
- net GNDREF: now also NT1.1
- new net GND1: NT1.2
Other:
- note added: "NetDie"
Changed lines of the file:
@@
 Sheet 6 7
 Title "Alimentación"
-Date "2021-03-03"
-Rev "1.0"
+Date "2021-03-30"
+Rev ""
 Comp "Crédito DyM de PCBs"
 Comment1 ""
@@
 $EndDescr
 $Comp
-L Regulator_Switching:LM2596S-5 U11
+L Regulator_Switching:LM2596S-5 U5
 U 1 1 603F9E77
 P 4100 4000
-F 0 "U11" H 4100 4367 50  0000 C CNN
+F 0 "U5" H 4100 4367 50  0000 C CNN
 F 1 "LM2596S-5" H 4100 4276 50  0000 C CNN
 F 2 "Package_TO_SOT_SMD:TO-263-5_TabPin3" H 4150 3750 50  0001 L CIN
@@
 $EndComp
 $Comp
-L power:+BATT #PWR075
+L power:+BATT #PWR069
 U 1 1 60401D05
 P 2900 3850
-F 0 "#PWR075" H 2900 3700 50  0001 C CNN
+F 0 "#PWR069" H 2900 3700 50  0001 C CNN
 F 1 "+BATT" H 2915 4023 50  0000 C CNN
 F 2 "" H 2900 3850 50  0001 C CNN
@@
 	5300 4500 5300 4450
 $Comp
-L power:+5V #PWR082
+L power:+5V #PWR076
 U 1 1 604017EE
 P 7500 3850
-F 0 "#PWR082" H 7500 3700 50  0001 C CNN
+F 0 "#PWR076" H 7500 3700 50  0001 C CNN
 F 1 "+5V" H 7515 4023 50  0000 C CNN
 F 2 "" H 7500 3850 50  0001 C CNN
@@
 $EndComp
 $Comp
-L power:+5V #PWR081
+L power:+5V #PWR075
 U 1 1 60401172
 P 5500 4050
-F 0 "#PWR081" H 5500 3900 50  0001 C CNN
+F 0 "#PWR075" H 5500 3900 50  0001 C CNN
 F 1 "+5V" H 5515 4223 50  0000 C CNN
 F 2 "" H 5500 4050 50  0001 C CNN
@@
 $EndComp
 $Comp
-L power:+3.3V #PWR085
+L power:+3.3V #PWR079
 U 1 1 6040099D
 P 8650 3850
-F 0 "#PWR085" H 8650 3700 50  0001 C CNN
+F 0 "#PWR079" H 8650 3700 50  0001 C CNN
 F 1 "+3.3V" H 8665 4023 50  0000 C CNN
 F 2 "" H 8650 3850 50  0001 C CNN
@@
 $EndComp
 $Comp
-L Regulator_Linear:AMS1117-3.3 U12
+L Regulator_Linear:AMS1117-3.3 U6
 U 1 1 603FAA46
 P 8100 3900
-F 0 "U12" H 8100 4142 50  0000 C CNN
+F 0 "U6" H 8100 4142 50  0000 C CNN
 F 1 "AMS1117-3.3" H 8100 4051 50  0000 C CNN
 F 2 "Package_TO_SOT_SMD:SOT-223-3_TabPin2" H 8100 4100 50  0001 C CNN
@@
 	8650 4300 8650 4250
 $Comp
-L power:GNDREF #PWR077
+L power:GNDREF #PWR071
 U 1 1 604290E2
 P 3550 4150
-F 0 "#PWR077" H 3550 3900 50  0001 C CNN
+F 0 "#PWR071" H 3550 3900 50  0001 C CNN
 F 1 "GNDREF" H 3555 3977 50  0000 C CNN
 F 2 "" H 3550 4150 50  0001 C CNN
@@
 $EndComp
 $Comp
-L power:GNDREF #PWR078
+L power:GNDREF #PWR072
 U 1 1 6042A132
 P 4100 4350
-F 0 "#PWR078" H 4100 4100 50  0001 C CNN
+F 0 "#PWR072" H 4100 4100 50  0001 C CNN
 F 1 "GNDREF" H 4105 4177 50  0000 C CNN
 F 2 "" H 4100 4350 50  0001 C CNN
@@
 $EndComp
 $Comp
-L power:GNDREF #PWR079
+L power:GNDREF #PWR073
 U 1 1 6042A56D
 P 4700 4500
-F 0 "#PWR079" H 4700 4250 50  0001 C CNN
+F 0 "#PWR073" H 4700 4250 50  0001 C CNN
 F 1 "GNDREF" H 4705 4327 50  0000 C CNN
 F 2 "" H 4700 4500 50  0001 C CNN
@@
 $EndComp
 $Comp
-L power:GNDREF #PWR080
+L power:GNDREF #PWR074
 U 1 1 6042AA6F
 P 5300 4500
-F 0 "#PWR080" H 5300 4250 50  0001 C CNN
+F 0 "#PWR074" H 5300 4250 50  0001 C CNN
 F 1 "GNDREF" H 5305 4327 50  0000 C CNN
 F 2 "" H 5300 4500 50  0001 C CNN
@@
 $EndComp
 $Comp
-L power:GNDREF #PWR083
+L power:GNDREF #PWR077
 U 1 1 6042AE3F
 P 7500 4350
-F 0 "#PWR083" H 7500 4100 50  0001 C CNN
+F 0 "#PWR077" H 7500 4100 50  0001 C CNN
 F 1 "GNDREF" H 7505 4177 50  0000 C CNN
 F 2 "" H 7500 4350 50  0001 C CNN
@@
 $EndComp
 $Comp
-L power:GNDREF #PWR084
+L power:GNDREF #PWR078
 U 1 1 6042B3F6
 P 8100 4250
-F 0 "#PWR084" H 8100 4000 50  0001 C CNN
+F 0 "#PWR078" H 8100 4000 50  0001 C CNN
 F 1 "GNDREF" H 8105 4077 50  0000 C CNN
 F 2 "" H 8100 4250 50  0001 C CNN
@@
 $EndComp
 $Comp
-L power:GNDREF #PWR086
+L power:GNDREF #PWR080
 U 1 1 6042B7F2
 P 8650 4300
-F 0 "#PWR086" H 8650 4050 50  0001 C CNN
+F 0 "#PWR080" H 8650 4050 50  0001 C CNN
 F 1 "GNDREF" H 8655 4127 50  0000 C CNN
 F 2 "" H 8650 4300 50  0001 C CNN
@@
 $EndComp
 $Comp
-L power:GNDREF #PWR076
+L power:GNDREF #PWR070
 U 1 1 6044FE03
 P 3000 4550
-F 0 "#PWR076" H 3000 4300 50  0001 C CNN
+F 0 "#PWR070" H 3000 4300 50  0001 C CNN
 F 1 "GNDREF" H 3005 4377 50  0000 C CNN
 F 2 "" H 3000 4550 50  0001 C CNN
@@
 3.3V Power Supply
 $Comp
-L Connector_Generic:Conn_01x02 J7
+L Connector_Generic:Conn_01x02 J13
 U 1 1 604A4B4C
 P 2500 4000
-F 0 "J7" H 2418 3675 50  0000 C CNN
+F 0 "J13" H 2418 3675 50  0000 C CNN
 F 1 "Batería2" H 2418 3766 50  0000 C CNN
 F 2 "Battery:BatteryHolder_MPD_BH-18650-PC2" H 2500 4000 50  0001 C CNN
@@
 $EndComp
 $Comp
-L Connector_Generic:Conn_01x02 J8
+L Connector_Generic:Conn_01x02 J14
 U 1 1 604A583E
 P 2500 4500
-F 0 "J8" H 2418 4175 50  0000 C CNN
+F 0 "J14" H 2418 4175 50  0000 C CNN
 F 1 "Bateria1" H 2418 4266 50  0000 C CNN
 F 2 "Battery:BatteryHolder_MPD_BH-18650-PC2" H 2500 4500 50  0001 C CNN
@@
 Wire Wire Line
 	2850 4100 3550 4100
+$Comp
+L Device:Net-Tie_2 NT1
+U 1 1 606F2102
+P 4100 2700
+F 0 "NT1" H 4100 2881 50  0000 C CNN
+F 1 "Net-Tie_2" H 4100 2790 50  0000 C CNN
+F 2 "NetTie:NetTie-2_SMD_Pad2.0mm" H 4100 2700 50  0001 C CNN
+F 3 "~" H 4100 2700 50  0001 C CNN
+	1    4100 2700
+	1    0    0    -1
+$EndComp
+$Comp
+L power:GND1 #PWR0101
+U 1 1 606F39DF
+P 4250 2750
+F 0 "#PWR0101" H 4250 2500 50  0001 C CNN
+F 1 "GND1" H 4255 2577 50  0000 C CNN
+F 2 "" H 4250 2750 50  0001 C CNN
+F 3 "" H 4250 2750 50  0001 C CNN
+	1    4250 2750
+	1    0    0    -1
+$EndComp
+$Comp
+L power:GNDREF #PWR0102
+U 1 1 606F3E87
+P 3950 2750
+F 0 "#PWR0102" H 3950 2500 50  0001 C CNN
+F 1 "GNDREF" H 3955 2577 50  0000 C CNN
+F 2 "" H 3950 2750 50  0001 C CNN
+F 3 "" H 3950 2750 50  0001 C CNN
+	1    3950 2750
+	1    0    0    -1
+$EndComp
+Wire Wire Line
+	4250 2750 4250 2700
+Wire Wire Line
+	4250 2700 4200 2700
+Wire Wire Line
+	3950 2750 3950 2700
+Wire Wire Line
+	3950 2700 4000 2700
+Text Notes 3700 2350 0    157  ~ 0
+NetDie
+Wire Notes Line width 10
+	4400 3000 3750 3000
+Wire Notes Line width 10
+	3750 3000 3750 2450
+Wire Notes Line width 10
+	3750 2450 4400 2450
+Wire Notes Line width 10
+	4400 2450 4400 3000
 $EndSCHEMATC
