File: Microcontrolador.sch (KiCad schematic (older format))
At the start: 32 parts, among them J4 USB, J5 SWD, J6 BOOT MODE, SW2 PID Init, SW3 RESET, U10 STM32F103C8Tx, Y1 8MHz

Commit message: Placa terminada
Parts:
- renumbered J4 to J10, J5 to J11, J6 to J12, U10 to U4
Connections:
- net +3V3: now also J12.5 (Pin_5); no longer J12.1 (Pin_1)
- net GNDREF: now also J12.1 (Pin_1), J12.2 (Pin_2); no longer J12.3 (Pin_3), J12.4 (Pin_4)
- net at R21.1: now also J12.3 (Pin_3); no longer J12.2 (Pin_2)
- net at R24.2: now also J12.4 (Pin_4); no longer J12.5 (Pin_5)
Other:
- moved on the sheet: R21, R24
