File: Puente H.sch (KiCad schematic (older format))
At the start: 6 parts, among them J1 Motor izquierda, J2 Motor derecha, U7 L9110, U8 L9110

Commit message: Placa terminada
Parts:
- renumbered J1 to J7, J2 to J8, U7 to U1, U8 to U2
Changed lines of the file:
@@
 Sheet 3 7
 Title "Puente H"
-Date "2021-03-03"
-Rev "1.0"
+Date "2021-03-30"
+Rev ""
 Comp "Crédito DyM de PCBs"
 Comment1 ""
@@
 $EndDescr
 $Comp
-L power:+5V #PWR027
+L power:+5V #PWR021
 U 1 1 6043E356
 P 5200 2950
-F 0 "#PWR027" H 5200 2800 50  0001 C CNN
+F 0 "#PWR021" H 5200 2800 50  0001 C CNN
 F 1 "+5V" H 5215 3123 50  0000 C CNN
 F 2 "" H 5200 2950 50  0001 C CNN
@@
 MOTIA
 $Comp
-L Mis_componentes:L9110 U8
+L Mis_componentes:L9110 U2
 U 1 1 6041FEF1
 P 5600 4900
-F 0 "U8" H 5600 5615 50  0000 C CNN
+F 0 "U2" H 5600 5615 50  0000 C CNN
 F 1 "L9110" H 5600 5524 50  0000 C CNN
 F 2 "Package_DIP:DIP-8_W7.62mm" H 5600 4900 50  0001 C CNN
@@
 $EndComp
 $Comp
-L power:GNDREF #PWR029
+L power:GNDREF #PWR023
 U 1 1 60431AED
 P 6000 3650
-F 0 "#PWR029" H 6000 3400 50  0001 C CNN
+F 0 "#PWR023" H 6000 3400 50  0001 C CNN
 F 1 "GNDREF" H 6005 3477 50  0000 C CNN
 F 2 "" H 6000 3650 50  0001 C CNN
@@
 $EndComp
 $Comp
-L power:GNDREF #PWR030
+L power:GNDREF #PWR024
 U 1 1 60431FB6
 P 6000 4800
-F 0 "#PWR030" H 6000 4550 50  0001 C CNN
+F 0 "#PWR024" H 6000 4550 50  0001 C CNN
 F 1 "GNDREF" H 6005 4627 50  0000 C CNN
 F 2 "" H 6000 4800 50  0001 C CNN
@@
 $EndComp
 $Comp
-L power:+5V #PWR028
+L power:+5V #PWR022
 U 1 1 6043DEAE
 P 5200 3950
-F 0 "#PWR028" H 5200 3800 50  0001 C CNN
+F 0 "#PWR022" H 5200 3800 50  0001 C CNN
 F 1 "+5V" H 5215 4123 50  0000 C CNN
 F 2 "" H 5200 3950 50  0001 C CNN
@@
 $EndComp
 $Comp
-L power:GNDREF #PWR025
+L power:GNDREF #PWR019
 U 1 1 604DDB80
 P 4750 3050
-F 0 "#PWR025" H 4750 2800 50  0001 C CNN
+F 0 "#PWR019" H 4750 2800 50  0001 C CNN
 F 1 "GNDREF" H 4755 2877 50  0000 C CNN
 F 2 "" H 4750 3050 50  0001 C CNN
@@
 $EndComp
 $Comp
-L power:GNDREF #PWR026
+L power:GNDREF #PWR020
 U 1 1 604DE047
 P 4800 4050
-F 0 "#PWR026" H 4800 3800 50  0001 C CNN
+F 0 "#PWR020" H 4800 3800 50  0001 C CNN
 F 1 "GNDREF" H 4805 3877 50  0000 C CNN
 F 2 "" H 4800 4050 50  0001 C CNN
@@
 	5100 3250 5250 3250
 $Comp
-L Mis_componentes:L9110 U7
+L Mis_componentes:L9110 U1
 U 1 1 6041F65F
 P 5600 3700
-F 0 "U7" H 5600 4415 50  0000 C CNN
+F 0 "U1" H 5600 4415 50  0000 C CNN
 F 1 "L9110" H 5600 4324 50  0000 C CNN
 F 2 "Package_DIP:DIP-8_W7.62mm" H 5600 3700 50  0001 C CNN
@@
 	5050 4550 5100 4550
 $Comp
-L Connector_Generic:Conn_01x02 J2
+L Connector_Generic:Conn_01x02 J8
 U 1 1 6043D24F
 P 4850 4550
-F 0 "J2" H 4850 4700 50  0000 C CNN
+F 0 "J8" H 4850 4700 50  0000 C CNN
 F 1 "Motor derecha" H 4850 4350 50  0000 C CNN
 F 2 "Connector_JST:JST_EH_B2B-EH-A_1x02_P2.50mm_Vertical" H 4850 4550 50  0001 C CNN
@@
 $EndComp
 $Comp
-L Connector_Generic:Conn_01x02 J1
+L Connector_Generic:Conn_01x02 J7
 U 1 1 6043CC3C
 P 4850 3450
-F 0 "J1" H 4850 3250 50  0000 C CNN
+F 0 "J7" H 4850 3250 50  0000 C CNN
 F 1 "Motor izquierda" H 4900 3550 50  0000 C CNN
 F 2 "Connector_JST:JST_EH_B2B-EH-A_1x02_P2.50mm_Vertical" H 4850 3450 50  0001 C CNN
