File: Sensores.sch (KiCad schematic (older format))
At the start: 18 parts, among them U1 TCRT5000, U2 TCRT5000, U3 TCRT5000, U4 TCRT5000, U5 TCRT5000, U6 TCRT5000

Commit message: Placa terminada
Parts:
- removed R10: 120R, Resistor_SMD:R_0805_2012Metric, symbol Device:R
- removed U1, U2, U3, U4, U5, U6: TCRT5000, Connector_PinSocket_2.54mm:PinSocket_2x02_P2.54mm_Vertical, symbol Mis_componentes:TCRT5000
- added J1: SENSOR 1, Mis_componentes:TCRT5000, symbol Connector_Generic:Conn_02x03_Odd_Even
- added J2: SENSOR 4, Mis_componentes:TCRT5000, symbol Connector_Generic:Conn_02x03_Odd_Even
- added J3: SENSOR 2, Mis_componentes:TCRT5000, symbol Connector_Generic:Conn_02x03_Odd_Even
- added J4: SENSOR 5, Mis_componentes:TCRT5000, symbol Connector_Generic:Conn_02x03_Odd_Even
- added J5: SENSOR 3, Mis_componentes:TCRT5000, symbol Connector_Generic:Conn_02x03_Odd_Even
- added J6: SENSOR 6, Mis_componentes:TCRT5000, symbol Connector_Generic:Conn_02x03_Odd_Even
- added R12: 120R, Resistor_SMD:R_0805_2012Metric, symbol Device:R
- R1, R2, R5, R6, R9: value 120R -> 50k
- R11, R3, R4, R7, R8: value 50k -> 120R
- renumbered R12 to R10
Connections:
- net +3V3: now also J1.1 (Pin_1), J1.5 (Pin_5), J2.1 (Pin_1), J2.5 (Pin_5), J3.1 (Pin_1), J3.5 (Pin_5), J4.1 (Pin_1), J4.5 (Pin_5), J5.1 (Pin_1), J5.5 (Pin_5), J6.1 (Pin_1), J6.5 (Pin_5)
- net GNDREF: now also R11.1, R3.1, R4.1, R7.1, R8.1, R12.1; no longer R11.2, R3.2, R4.2, R7.2, R8.2
- net SENSOR1: now also R1.1, J1.6 (Pin_6); no longer R3.1
- net SENSOR2: now also R5.1, J3.6 (Pin_6); no longer R7.1
- net SENSOR3: now also R9.1, J5.6 (Pin_6); no longer R11.1
- net SENSOR4: now also R2.1, J2.6 (Pin_6); no longer R4.1
- net SENSOR5: now also R6.1, J4.6 (Pin_6); no longer R8.1
- net SENSOR6: now also J6.6 (Pin_6)
- new net: J6.2 (Pin_2), R12.2
- new net: J4.2 (Pin_2), R8.2
- new net: J2.2 (Pin_2), R4.2
- new net: J5.2 (Pin_2), R11.2
- new net: J3.2 (Pin_2), R7.2
- new net: J1.2 (Pin_2), R3.2
